File: Wand/Wand.sch (KiCad schematic (older format))
At the start: 20 parts, among them P1 ISP, P2 KLB4, P3 BASE, U1 ATMEGA328-MMH, U2 MAX31855KASA+, U3 MPU-6050

Commit message: Initial re-layout of the Hotstick Wand.
- Fixed tip connector
- Fixed the vias under the MPU-6050
- Changed to use an op-amp to read the tip temp
Parts:
- removed U2: MAX31855KASA+, Housings_SOIC:SOIC-8_3.9x4.9mm_Pitch1.27mm, symbol MAX6675
- added C3, C8: 100n, Capacitors_SMD:C_0402, symbol C
- added R1: 1M, Resistors_SMD:R_0402, symbol R
- added R10: 56K, Resistors_SMD:R_0402, symbol R
- added R11, R8: 1K, Resistors_SMD:R_0402, symbol R
- added R9: 100R, Resistors_SMD:R_0402, symbol R
- added U2: OPA336, TO_SOT_Packages_SMD:SOT-23-5, symbol OPA336
Connections:
- net labels added: TEMP
- net labels removed: TIP_TEMP_SELECT
- wire segments 98 -> 107
Other:
- moved on the sheet: D1, D2, R4, R5, R6, R7
